Commit message: Update config.

File: pca9685_ros2_control/description.urdf.xacro (robot description, xacro)
@@ -1,51 +1,23 @@
 <?xml version="1.0"?>
 <robot xmlns:xacro="http://www.ros.org/wiki/xacro" name="pca9685_example">
-  <link name="base_link"/>
-  <joint name="joint3" type="continuous">
-    <origin xyz="0.25 0.25 0.0" rpy="0 0 3.141"/>
-    <parent link="base_link"/>
-    <child link="front_left_wheel"/>
-  </joint>
-  <link name="front_left_wheel"/>
-  <joint name="joint1" type="continuous">
-    <origin xyz="0.25 -0.25 0.0" rpy="0 0 0"/>
-    <parent link="base_link"/>
-    <child link="front_right_wheel"/>
-  </joint>
-  <link name="front_right_wheel"/>
-  <!-- <joint name="back_left_joint" type="continuous">
-    <origin xyz="-0.25 0.25 0.0" rpy="0 0 0"/>
-    <parent link="base_link"/>
-    <child link="back_left_wheel"/>
-    <axis xyz="0 0 1"/>
-  </joint>
-  <link name="back_left_wheel"/>
-  <joint name="back_right_joint" type="continuous">
-    <origin xyz="-0.25 -0.25 0.0" rpy="0 0 0"/>
-    <parent link="base_link"/>
-    <child link="back_right_wheel"/>
-    <axis xyz="0 0 1"/>
-  </joint>
-  <link name="back_right_wheel"/> -->
   <ros2_control name="pca9685_ros2_control_example" type="system">
     <hardware>
       <plugin>pca9685_hardware_interface/Pca9685SystemHardware</plugin>
     </hardware>
-    <joint name="joint0">
+    <joint name="joint_0">
       <command_interface name="velocity"/>
       <state_interface name="velocity"/>
     </joint>
-    <joint name="joint1">
+    <joint name="joint_1">
       <command_interface name="velocity"/>
       <state_interface name="velocity"/>
     </joint>
-    <joint name="joint2">
+    <joint name="joint_2">
       <command_interface name="velocity"/>
       <state_interface name="velocity"/>
     </joint>
-    <joint name="joint3">
+    <joint name="joint_3">
       <command_interface name="velocity"/>
       <state_interface name="velocity"/>
-      <axis xyz="-1 0 0"/>
     </joint>
     <joint name="joint_4">
